Commit message: UpperBodyXo URDF
need to add robotPose to urdf. Put into SCS

File: RobotModels/createdSDFURDF/athena_v1_robot.urdf (robot description, URDF)
Before this commit: robot athena_v1, 13 links, 12 joints
Joints:
- joint ll1_hip_yaw: axis (none) -> 0 0 0
- joint ll2_hip_rol: axis (none) -> 0 0 0
- joint ll3_hip_pit: axis (none) -> 0 0 0
- joint ll4_kne_pit: axis (none) -> 0 0 0
- joint ll5_ank_pit: axis (none) -> 0 0 0
- joint ll6_ank_rol: axis (none) -> 0 0 0
- joint rl1_hip_yaw: axis (none) -> 0 0 0
- joint rl2_hip_rol: axis (none) -> 0 0 0
- joint rl3_hip_pit: axis (none) -> 0 0 0
- joint rl4_kne_pit: axis (none) -> 0 0 0
- joint rl5_ank_pit: axis (none) -> 0 0 0
- joint rl6_ank_rol: axis (none) -> 0 0 0
